File: Circuito/PCB_Univ_V0.sch (EAGLE design)
At the start: 21 parts

Commit message: Circuito V0
Parts:
- removed C2: 100uF, DAIMOB:CAP_SMD_100U
- removed C3: 100nF, rcl2:C-EUC1206
- removed R1: 4.7k, rcl:R-EU_R1206
- removed R2: (no value), rcl:R-EU_R1206
- removed R3: 10k, rcl:R-EU_R1206
- removed U$10: SW_SMD, DAIMOB:SW_SMD
- removed U$11, U$12: JP_SMD, DAIMOB:JP_SMD
- removed U$3: RFM95W, DAIMOB:RFM95W
- removed U$4: MCP1826S-3302E/DB, DAIMOB:MCP1826S-3302E/DB
- removed U$5: PMV250EPA, DAIMOB:PMV250EPA
- removed U$6: SWITCH_SMD, DAIMOB:SWITCH_SMD
- removed U$7: ANTENA_IPX, DAIMOB:ANTENA_IPX
- removed U$8: CHARGER, DAIMOB:CHARGER
- removed U$9: RTC_DS3231, DAIMOB:RTC_DS3231
- removed X1: (no value), con-ptr500:AK500/2
- removed X2: (no value), con-ptr500:AK500/12
- removed X4: (no value), con-ptr500:AK500/3
- added ESP1: ESP12_MOD, DAIMOB:ESP12_MOD
- added JP1: (no value), pinhead:PINHD-1X17
- added JP2: (no value), pinhead:PINHD-1X14
- C1: value 100uF -> (none); device DAIMOB:CAP_SMD_100U -> rcl2:CPOL-EUE3.5-8
- U$1: value PRO_MINI -> DRIVER_MOTOR; device DAIMOB:PRO_MINI -> DAIMOB:DRIVER_MOTOR
- U$2: value TPL5110 -> DRIVER_MOTOR; device DAIMOB:TPL5110 -> DAIMOB:DRIVER_MOTOR
Connections:
- removed net 0V: U$8.IN-, X1-1.KL
- removed net 5V: U$8.IN+, X1-2.KL
- removed net A0: U$1.A0, X2-10.KL
- removed net A1: U$1.A1, X2-9.KL
- removed net A2: U$1.A2, X2-8.KL
- removed net ANT: U$3.ANT, U$7.SENAL
- removed net BAT+: U$8.B+, X2-1.KL
- removed net BAT-: U$8.B-, X2-2.KL
- removed net DELAY: R2.2, U$10.3, U$10.4, U$2.DELAY
- removed net DONE: R3.2, U$1.4, U$2.DONE
- removed net DRV: U$2.DRV, U$5.G
- removed net EN: U$12.P$2, U$2.EN
- removed net GPIO0: U$1.3, U$3.DIO0
- removed net IO5: U$1.5, X2-3.KL
- removed net IO6: U$1.6, X2-4.KL
- removed net IO7: U$1.7, X2-5.KL
- removed net IO8: U$1.8, X2-7.KL
- removed net MISO: U$1.12, U$3.MISO
- removed net MOSI: U$1.11, U$3.MOSI
- removed net NSS: U$1.10, U$3.NSS
- removed net OUT+: U$6.1, U$8.OUT+
- removed net OUT+1: U$11.P$2, U$6.2
- removed net RST: U$1.2, U$3.RST
- removed net SCK: U$1.13, U$3.SCK
- removed net SCL: U$1.A5, U$9.SCL, X4-3.KL
- removed net SDA: U$1.A4, U$9.SDA, X4-2.KL
- removed net TEMP: R1.1, U$1.9, X2-6.KL
- removed net VDD: C3.1, U$10.1, U$10.2, U$11.P$3, U$12.P$3, U$2.VDD, U$5.S
- removed net VIN: C1.+, U$11.P$1, U$4.IN, U$5.D
- new net N$1: ESP1.P27, U$1.N1
- new net N$10: ESP1.P33, JP2.7
- new net N$11: ESP1.P32, JP2.8
- new net N$12: ESP1.P35, JP2.9
- new net N$13: ESP1.P34, JP2.10
- new net N$14: ESP1.SVN, JP2.11
- new net N$15: ESP1.SVP, JP2.12
- new net N$16: ESP1.EN, JP2.13
- new net N$17: ESP1.3V, JP2.14
- new net N$18: ESP1.P23, JP1.1
- new net N$19: ESP1.P22, JP1.2
- new net N$2: ESP1.P26, U$1.N2
- new net N$20: ESP1.TX, JP1.3
- new net N$21: ESP1.RX, JP1.4
- new net N$22: ESP1.P21, JP1.5
- new net N$23: ESP1.P19, JP1.6
- new net N$24: ESP1.P18, JP1.7
- new net N$25: ESP1.P5, JP1.8
- new net N$26: ESP1.P17, JP1.9
- new net N$27: ESP1.P16, JP1.10
- new net N$28: ESP1.P4, JP1.11
- new net N$29: ESP1.P0, JP1.12
- new net N$3: ESP1.P14, U$1.ENA
- new net N$30: ESP1.P2, JP1.13
- new net N$31: ESP1.P15, JP1.14
- new net N$32: ESP1.SD1, JP1.15
- new net N$33: ESP1.SDO, JP1.16
- new net N$34: ESP1.CLK, JP1.17
- new net N$4: ESP1.CMD, JP2.1
- new net N$5: ESP1.SD3, JP2.2
- new net N$6: ESP1.SD2, JP2.3
- new net N$7: ESP1.P13, JP2.4
- new net N$8: ESP1.P12, JP2.5
- new net N$9: ESP1.P25, JP2.6
- net GND: now also ESP1.GND, ESP1.GND@1, ESP1.GND@2; no longer C2.-, C3.2, R2.1, R3.1, U$1.GND@1, U$12.P$1, U$3.GND, U$3.GND@1, U$3.GND@2, U$4.GND, U$4.GND@1, U$7.GND, U$7.GND@1, U$7.GND@2, U$8.OUT-, U$9.GND, U$9.GND@1, X2-11.KL, X2-12.KL
- net VCC: now also C1.+, ESP1.5V, U$1.5V, U$2.5V; no longer C2.+, R1.2, U$1.VCC, U$3.3.3V, U$4.OUT, U$9.VCC, X4-1.KL
Other:
- note removed: "DIO0"
- note removed: "miso"
- note removed: "mosi"
- note removed: "nss"
- note removed: "rstLora"
- note removed: "sck"
- moved on the sheet: C1
